File: examples/fc/power.kicad_sch (KiCad schematic)
At the start: 14 parts, among them J1 VBAT 2-6S, U1 TPS54302, U2 AP2112K-3.3

Commit message: Add structured schematic scenes and fix example overlaps
Other:
- moved on the sheet: C3
Changed lines of the file:
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@@
 		(dnp no)
 		(property "Reference" "U1"
-			(at 106.68 72.39 0)
-			(effects
-				(font
-					(size 1.27 1.27)
-				)
+			(at 91.44 90.17 0)
+			(effects
+				(font
+					(size 1.27 1.27)
+				)
+				(justify left)
 			)
 		)
 		(property "Value" "TPS54302"
-			(at 106.68 90.17 0)
-			(effects
-				(font
-					(size 1.27 1.27)
-				)
+			(at 91.44 92.71 0)
+			(effects
+				(font
+					(size 1.27 1.27)
+				)
+				(justify left)
 			)
 		)
@@
 	(symbol
 		(lib_id "Device:C")
-		(at 140.97 87.63 0)
+		(at 151.13 87.63 0)
 		(unit 1)
 		(exclude_from_sim no)
@@
 		(dnp no)
 		(property "Reference" "C3"
-			(at 144.272 86.36 0)
+			(at 154.432 86.36 0)
 			(effects
 				(font
@@
 		)
 		(property "Value" "22u"
-			(at 144.272 88.9 0)
-			(effects
-				(font
-					(size 1.27 1.27)
-				)
-				(justify left)
-			)
-		)
-		(property "Footprint" ""
-			(at 140.97 87.63 0)
+			(at 154.432 88.9 0)
+			(effects
+				(font
+					(size 1.27 1.27)
+				)
+				(justify left)
+			)
+		)
+		(property "Footprint" ""
+			(at 151.13 87.63 0)
 			(effects
 				(font
@@
 	(symbol
 		(lib_id "power:+5V")
-		(at 151.13 73.66 0)
+		(at 161.29 73.66 0)
 		(unit 1)
 		(exclude_from_sim no)
@@
 		(dnp no)
 		(property "Reference" "#PWR0001"
-			(at 153.162 72.39 0)
+			(at 163.322 72.39 0)
 			(effects
 				(font
@@
 		)
 		(property "Value" "+5V"
-			(at 153.162 74.93 0)
-			(effects
-				(font
-					(size 1.27 1.27)
-				)
-				(justify left)
-			)
-		)
-		(property "Footprint" ""
-			(at 151.13 73.66 0)
+			(at 163.322 74.93 0)
+			(effects
+				(font
+					(size 1.27 1.27)
+				)
+				(justify left)
+			)
+		)
+		(property "Footprint" ""
+			(at 161.29 73.66 0)
 			(effects
 				(font
@@
 		(dnp no)
 		(property "Reference" "U2"
-			(at 170.18 104.775 0)
-			(effects
-				(font
-					(size 1.27 1.27)
-				)
+			(at 176.53 96.52 0)
+			(effects
+				(font
+					(size 1.27 1.27)
+				)
+				(justify left)
 			)
 		)
 		(property "Value" "AP2112K-3.3"
-			(at 170.18 121.92 0)
-			(effects
-				(font
-					(size 1.27 1.27)
-				)
+			(at 176.53 99.06 0)
+			(effects
+				(font
+					(size 1.27 1.27)
+				)
+				(justify left)
 			)
 		)
@@
 	(symbol
 		(lib_id "power:+5V")
-		(at 137.16 165.1 0)
+		(at 147.32 165.1 0)
 		(unit 1)
 		(exclude_from_sim no)
@@
 		(dnp no)
 		(property "Reference" "#PWR0002"
-			(at 139.192 163.83 0)
+			(at 149.352 163.83 0)
 			(effects
 				(font
@@
 		)
 		(property "Value" "+5V"
-			(at 139.192 166.37 0)
-			(effects
-				(font
-					(size 1.27 1.27)
-				)
-				(justify left)
-			)
-		)
-		(property "Footprint" ""
-			(at 137.16 165.1 0)
+			(at 149.352 166.37 0)
+			(effects
+				(font
+					(size 1.27 1.27)
+				)
+				(justify left)
+			)
+		)
+		(property "Footprint" ""
+			(at 147.32 165.1 0)
 			(effects
 				(font
@@
 	(symbol
 		(lib_id "power:GND")
-		(at 99.06 165.1 0)
+		(at 109.22 165.1 0)
 		(unit 1)
 		(exclude_from_sim no)
@@
 		(dnp no)
 		(property "Reference" "#PWR0003"
-			(at 101.6 163.83 0)
+			(at 111.76 163.83 0)
 			(effects
 				(font
@@
 		)
 		(property "Value" "GND"
-			(at 101.6 166.37 0)
-			(effects
-				(font
-					(size 1.27 1.27)
-				)
-				(justify left)
-			)
-		)
-		(property "Footprint" ""
-			(at 99.06 165.1 0)
+			(at 111.76 166.37 0)
+			(effects
+				(font
+					(size 1.27 1.27)
+				)
+				(justify left)
+			)
+		)
+		(property "Footprint" ""
+			(at 109.22 165.1 0)
 			(effects
 				(font
@@
 	(symbol
 		(lib_id "power:GND")
-		(at 140.97 96.52 0)
+		(at 151.13 96.52 0)
 		(unit 1)
 		(exclude_from_sim no)
@@
 		(dnp no)
 		(property "Reference" "#PWR0007"
-			(at 143.51 95.25 0)
+			(at 153.67 95.25 0)
 			(effects
 				(font
@@
 		)
 		(property "Value" "GND"
-			(at 143.51 97.79 0)
-			(effects
-				(font
-					(size 1.27 1.27)
-				)
-				(justify left)
-			)
-		)
-		(property "Footprint" ""
-			(at 140.97 96.52 0)
+			(at 153.67 97.79 0)
+			(effects
+				(font
+					(size 1.27 1.27)
+				)
+				(justify left)
+			)
+		)
+		(property "Footprint" ""
+			(at 151.13 96.52 0)
 			(effects
 				(font
@@
 		(pts
 			(xy 133.35 80.01)
-			(xy 140.97 80.01)
-		)
-		(stroke
-			(width 0)
-			(type default)
-		)
-	)
-	(wire
-		(pts
-			(xy 140.97 80.01)
-			(xy 140.97 83.82)
-		)
-		(stroke
-			(width 0)
-			(type default)
-		)
-	)
-	(wire
-		(pts
 			(xy 151.13 80.01)
-			(xy 151.13 73.66)
-		)
-		(stroke
-			(width 0)
-			(type default)
-		)
-	)
-	(wire
-		(pts
-			(xy 140.97 80.01)
+		)
+		(stroke
+			(width 0)
+			(type default)
+		)
+	)
+	(wire
+		(pts
 			(xy 151.13 80.01)
+			(xy 151.13 83.82)
+		)
+		(stroke
+			(width 0)
+			(type default)
+		)
+	)
+	(wire
+		(pts
+			(xy 161.29 80.01)
+			(xy 161.29 73.66)
+		)
+		(stroke
+			(width 0)
+			(type default)
+		)
+	)
+	(wire
+		(pts
+			(xy 151.13 80.01)
+			(xy 161.29 80.01)
 		)
 		(stroke
@@
 		(pts
 			(xy 127 165.1)
-			(xy 137.16 165.1)
+			(xy 147.32 165.1)
 		)
 		(stroke
@@
 		(pts
 			(xy 88.9 165.1)
-			(xy 99.06 165.1)
+			(xy 109.22 165.1)
 		)
 		(stroke
@@
 	(wire
 		(pts
-			(xy 140.97 91.44)
-			(xy 140.97 96.52)
-		)
-		(stroke
+			(xy 151.13 91.44)
+			(xy 151.13 96.52)
+		)
+		(stroke
