File: examples/esc4in1/esc4in1.kicad_sch (KiCad schematic)
At the start: 7 parts, among them J1 VBAT+, J2 VBAT-, J3 FC / DSHOT

Commit message: Improve PCB connectivity facts and ESC reference
Use native KiCad connectivity for point and unrouted inspection, set the advisory grid to 0.1 mm, and correct the ESC example's Betaflight connector pinout and partial routing. The ESC remains a non-operable reference with 74 unrouted connections; its schematic marks missing controller support circuits.
Connections:
- net +3V3: no longer J3.7 (Pin_7)
- net GND: now also J3.2 (Pin_2); no longer J3.8 (Pin_8)
- net Motor 1/DSHOT1: now also J3.5 (Pin_5); no longer J3.1 (Pin_1)
- net Motor 2/DSHOT2: now also J3.6 (Pin_6); no longer J3.2 (Pin_2)
- net Motor 3/DSHOT3: now also J3.7 (Pin_7); no longer J3.3 (Pin_3)
- net Motor 4/DSHOT4: now also J3.8 (Pin_8); no longer J3.4 (Pin_4)
- net VBAT: now also J3.1 (Pin_1); no longer J3.6 (Pin_6)
- no-connect marks 1 -> 2
Other:
- note added: "Betaflight ESC: 1 VBAT, 2 GND, 3 CURRENT NC, 4 TELEMETRY NC, 5-8 M1-M4"
- note added: "NOT OPERABLE: controller regulator, protection and sensing circuits incomplete"
Changed lines of the file:
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@@
 	(symbol
 		(lib_id "power:GND")
-		(at 40.64 58.42 0)
+		(at 55.88 58.42 0)
 		(unit 1)
 		(exclude_from_sim no)
@@
 		(dnp no)
 		(property "Reference" "#PWR0002"
-			(at 43.18 57.15 0)
+			(at 58.42 57.15 0)
 			(effects
 				(font
@@
 		)
 		(property "Value" "GND"
-			(at 43.18 59.69 0)
+			(at 58.42 59.69 0)
 			(effects
 				(font
@@
 		)
 		(property "Footprint" ""
-			(at 40.64 58.42 0)
+			(at 55.88 58.42 0)
 			(effects
 				(font
@@
 	(wire
 		(pts
+			(xy 48.26 63.5)
+			(xy 48.26 78.74)
+		)
+		(stroke
+			(width 0)
+			(type default)
+		)
+	)
+	(wire
+		(pts
+			(xy 48.26 78.74)
+			(xy 85.09 78.74)
+		)
+		(stroke
+			(width 0)
+			(type default)
+		)
+	)
+	(wire
+		(pts
+			(xy 45.72 63.5)
+			(xy 45.72 106.68)
+		)
+		(stroke
+			(width 0)
+			(type default)
+		)
+	)
+	(wire
+		(pts
+			(xy 45.72 106.68)
+			(xy 85.09 106.68)
+		)
+		(stroke
+			(width 0)
+			(type default)
+		)
+	)
+	(wire
+		(pts
+			(xy 43.18 63.5)
+			(xy 43.18 134.62)
+		)
+		(stroke
+			(width 0)
+			(type default)
+		)
+	)
+	(wire
+		(pts
+			(xy 43.18 134.62)
+			(xy 85.09 134.62)
+		)
+		(stroke
+			(width 0)
+			(type default)
+		)
+	)
+	(wire
+		(pts
+			(xy 40.64 63.5)
+			(xy 40.64 162.56)
+		)
+		(stroke
+			(width 0)
+			(type default)
+		)
+	)
+	(wire
+		(pts
+			(xy 40.64 162.56)
+			(xy 85.09 162.56)
+		)
+		(stroke
+			(width 0)
+			(type default)
+		)
+	)
+	(wire
+		(pts
 			(xy 58.42 63.5)
-			(xy 58.42 78.74)
-		)
-		(stroke
-			(width 0)
-			(type default)
-		)
-	)
-	(wire
-		(pts
-			(xy 58.42 78.74)
-			(xy 85.09 78.74)
-		)
-		(stroke
-			(width 0)
-			(type default)
-		)
-	)
-	(wire
-		(pts
-			(xy 55.88 63.5)
-			(xy 55.88 106.68)
-		)
-		(stroke
-			(width 0)
-			(type default)
-		)
-	)
-	(wire
-		(pts
-			(xy 55.88 106.68)
-			(xy 85.09 106.68)
-		)
-		(stroke
-			(width 0)
-			(type default)
-		)
-	)
-	(wire
-		(pts
-			(xy 53.34 63.5)
-			(xy 53.34 134.62)
-		)
-		(stroke
-			(width 0)
-			(type default)
-		)
-	)
-	(wire
-		(pts
-			(xy 53.34 134.62)
-			(xy 85.09 134.62)
-		)
-		(stroke
-			(width 0)
-			(type default)
-		)
-	)
-	(wire
-		(pts
-			(xy 50.8 63.5)
-			(xy 50.8 162.56)
-		)
-		(stroke
-			(width 0)
-			(type default)
-		)
-	)
-	(wire
-		(pts
-			(xy 50.8 162.56)
-			(xy 85.09 162.56)
-		)
-		(stroke
-			(width 0)
-			(type default)
-		)
-	)
-	(wire
-		(pts
-			(xy 45.72 63.5)
-			(xy 45.72 57.15)
-		)
-		(stroke
-			(width 0)
-			(type default)
-		)
-	)
-	(wire
-		(pts
-			(xy 43.18 63.5)
-			(xy 43.18 57.15)
+			(xy 58.42 57.15)
 		)
 		(stroke
@@
 	(wire
 		(pts
-			(xy 40.64 63.5)
-			(xy 40.64 58.42)
+			(xy 55.88 63.5)
+			(xy 55.88 58.42)
 		)
 		(stroke
@@
 	(global_label "VBAT"
 		(shape input)
-		(at 45.72 57.15 90)
-		(effects
-			(font
-				(size 1.27 1.27)
-			)
-			(justify left)
-		)
-	)
-	(global_label "+3V3"
-		(shape input)
-		(at 43.18 57.15 90)
+		(at 58.42 57.15 90)
 		(effects
 			(font
@@
 	)
 	(no_connect
-		(at 48.26 63.5)
+		(at 53.34 63.5)
+	)
+	(no_connect
+		(at 50.8 63.5)
 	)
 	(junction
@@
 	(text "AM32 target required; DShot signal is bidirectional"
 		(exclude_from_sim no)
-		(at 88.9 195.58 0)
+		(at 172.72 55.88 0)
 		(effects
 			(font
+				(size 1.27 1.27)
+				(thickness 0.254)
+			)
+			(justify left bottom)
+		)
+	)
+	(text "Betaflight ESC: 1 VBAT, 2 GND, 3 CURRENT NC, 4 TELEMETRY NC, 5-8 M1-M4"
+		(exclude_from_sim no)
+		(at 172.72 63.5 0)
+		(effects
+			(font
+				(size 1.27 1.27)
+				(thickness 0.254)
+			)
+			(justify left bottom)
+		)
+	)
+	(text "NOT OPERABLE: controller regulator, protection and sensing circuits incomplete"
+		(exclude_from_sim no)
+		(at 172.72 71.12 0)
+		(effects
+			(font
